Commit message: adding a joint and a position broadcaster package

File: src/cbot/cbot_description/urdf/j2s7s300.xacro (robot description, xacro)
@@ -44,5 +44,5 @@
     <xacro:property name="joint_base_type" value="fixed" />
     <xacro:property name="joint_base_axis_xyz" value="0 0 0" />
-    <xacro:property name="joint_base_origin_xyz" value="0 0 0.25" />
+    <xacro:property name="joint_base_origin_xyz" value="0 0 0" />
     <xacro:property name="joint_base_origin_rpy" value="0 0 0" />
     <xacro:property name="joint_1" value="joint_1" />

File: src/cbot/cbot_description/urdf/j2s7s300_standalone.xacro (robot description, xacro)
@@ -17,12 +17,29 @@
   <xacro:include filename="$(find cbot_description)/urdf/volta.urdf.xacro" />
   <xacro:include filename="$(find cbot_description)/urdf/j2s7s300.xacro"/>
+<link name="dummy_link">
+    <visual>
+      <geometry>
+        <cylinder length="0.1" radius="0.05"/>
+      </geometry>
+      <material name="blue"/>
+    </visual>
+    <collision>
+      <geometry>
+        <cylinder length="0.1" radius="0.05"/>
+      </geometry>
+    </collision>
+    <inertial>
+      <mass value="1"/>
+      <inertia ixx="1.0" ixy="0.0" ixz="0.0" iyy="1.0" iyz="0.0" izz="1.0"/>
+    </inertial>
+  </link>
   <!-- for gazebo -->
-  <link name="ground"/>
-  <joint name="connect_base_and_ground" type="fixed">
-    <child link="base_link" />
-    <parent link="ground" />
+  <joint name="connect_base_and_dummy" type="fixed">
+    <child link="dummy_link" />
+    <parent link="base_link" />
+    <origin xyz="0 0 0.251" rpy="0.0 0.0 0" />
   </joint>
   <xacro:volta_robot/>
-  <xacro:property name="robot_root" value="base_link" />
+  <xacro:property name="robot_root" value="dummy_link" />
   <xacro:j2s7s300  base_parent="${robot_root}"/>
 <!--
